File: locker_unit.sch (EAGLE design)
At the start: 30 parts, among them IC2 7805T, J1 RJ11, J2 RJ11, Q2 8 MHz, Q4 BC547, U1 PIC16F1705-X/PDIP

Commit message: Edit whole layout, add external LED header. Should be the final version.
Parts:
- removed LED1: RED, SparkFun-LED:LED5MM
- removed LED2: GREEN, SparkFun-LED:LED5MM
- removed R2: 220, SparkFun-Passives:RESISTORAXIAL-0.3
- added X3: (no value), Locker-custom:KK-156-2
- Q2: device crystal:CRYSTALHC49U70 -> SparkFun-FreqCtrl:CRYSTALHC49US
Connections:
- removed net N$7: LED2.C, R5.2
- net GND: no longer R2.1, R5.1
- net N$12: now also X3-2.S; no longer LED2.A
- net N$2: now also R5.1; no longer LED1.A
- net N$5: now also R5.2, X3-1.S; no longer LED1.C, R2.2
Changed lines of the file:
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@@
 <part name="GND6" library="SparkFun-Aesthetics" deviceset="GND" device=""/>
 <part name="GND7" library="SparkFun-Aesthetics" deviceset="GND" device=""/>
-<part name="Q2" library="crystal" deviceset="CRYSTAL" device="HC49U70" value="8 MHz"/>
+<part name="Q2" library="SparkFun-FreqCtrl" deviceset="CRYSTAL" device="HC49US" value="8 MHz"/>
 <part name="C3" library="rcl" deviceset="C-EU" device="025-025X050" value="22 pF"/>
 <part name="C4" library="rcl" deviceset="C-EU" device="025-025X050" value="22 pF"/>
@@
 <part name="SUPPLY9" library="SparkFun-Aesthetics" deviceset="5V" device=""/>
 <part name="Q4" library="SparkFun-DiscreteSemi" deviceset="TRANSISTOR_NPN" device="BC547" value="BC547"/>
-<part name="LED1" library="SparkFun-LED" deviceset="LED" device="5MM" value="RED"/>
-<part name="LED2" library="SparkFun-LED" deviceset="LED" device="5MM" value="GREEN"/>
-<part name="R2" library="SparkFun-Passives" deviceset="RESISTOR" device="AXIAL-0.3" value="220"/>
 <part name="R5" library="SparkFun-Passives" deviceset="RESISTOR" device="AXIAL-0.3" value="220"/>
-<part name="GND8" library="SparkFun-Aesthetics" deviceset="GND" device=""/>
-<part name="GND10" library="SparkFun-Aesthetics" deviceset="GND" device=""/>
 <part name="IC2" library="linear" deviceset="78*" device="T" technology="05" value="7805T"/>
 <part name="C9" library="rcl" deviceset="C-EU" device="050-030X075" value="0.1 uF"/>
@@
 <part name="X2" library="Locker-custom" deviceset="KK-156-2" device=""/>
 <part name="D2" library="diode" deviceset="1N4004" device=""/>
+<part name="X3" library="Locker-custom" deviceset="KK-156-2" device=""/>
 </parts>
 <sheets>
@@
 <instance part="SUPPLY9" gate="G$1" x="226.06" y="170.18"/>
 <instance part="Q4" gate="G$1" x="223.52" y="121.92"/>
-<instance part="LED1" gate="G$1" x="74.93" y="90.17"/>
-<instance part="LED2" gate="G$1" x="64.77" y="90.17"/>
-<instance part="R2" gate="G$1" x="74.93" y="78.74" rot="R90"/>
 <instance part="R5" gate="G$1" x="64.77" y="78.74" rot="R90"/>
-<instance part="GND8" gate="1" x="74.93" y="69.85"/>
-<instance part="GND10" gate="1" x="64.77" y="69.85"/>
 <instance part="IC2" gate="A1" x="35.56" y="160.02"/>
 <instance part="C9" gate="G$1" x="132.08" y="114.3" rot="R90"/>
@@
 <instance part="X2" gate="-2" x="260.35" y="153.67"/>
 <instance part="D2" gate="1" x="254" y="152.4" rot="R90"/>
+<instance part="X3" gate="-1" x="67.31" y="89.408"/>
+<instance part="X3" gate="-2" x="67.31" y="91.948"/>
 </instances>
 <busses>
@@
 </segment>
 <segment>
-<pinref part="R2" gate="G$1" pin="1"/>
-<pinref part="GND8" gate="1" pin="GND"/>
-<wire x1="74.93" y1="73.66" x2="74.93" y2="72.39" width="0.1524" layer="91"/>
-</segment>
-<segment>
-<pinref part="GND10" gate="1" pin="GND"/>
-<pinref part="R5" gate="G$1" pin="1"/>
-<wire x1="64.77" y1="73.66" x2="64.77" y2="72.39" width="0.1524" layer="91"/>
-</segment>
-<segment>
 <pinref part="GND12" gate="1" pin="GND"/>
 <pinref part="Q4" gate="G$1" pin="E"/>
@@
 </segment>
 </net>
-<net name="N$5" class="0">
-<segment>
-<pinref part="LED1" gate="G$1" pin="C"/>
-<pinref part="R2" gate="G$1" pin="2"/>
-<wire x1="74.93" y1="85.09" x2="74.93" y2="83.82" width="0.1524" layer="91"/>
-</segment>
-</net>
-<net name="N$7" class="0">
-<segment>
-<pinref part="R5" gate="G$1" pin="2"/>
-<pinref part="LED2" gate="G$1" pin="C"/>
-<wire x1="64.77" y1="85.09" x2="64.77" y2="83.82" width="0.1524" layer="91"/>
-</segment>
-</net>
 <net name="N$12" class="0">
 <segment>
 <pinref part="U1" gate="U1" pin="RA4/AN3/*T1G/OSC2/CLKOUT"/>
 <wire x1="91.44" y1="97.79" x2="64.77" y2="97.79" width="0.1524" layer="91"/>
-<pinref part="LED2" gate="G$1" pin="A"/>
-<wire x1="64.77" y1="97.79" x2="64.77" y2="92.71" width="0.1524" layer="91"/>
+<pinref part="X3" gate="-2" pin="S"/>
+<wire x1="64.77" y1="91.948" x2="64.77" y2="97.79" width="0.1524" layer="91"/>
 </segment>
 </net>
@@
 <segment>
 <pinref part="U1" gate="U1" pin="RC5/CCP1/RX"/>
-<pinref part="LED1" gate="G$1" pin="A"/>
-<wire x1="91.44" y1="92.71" x2="74.93" y2="92.71" width="0.1524" layer="91"/>
+<wire x1="91.44" y1="92.71" x2="73.66" y2="92.71" width="0.1524" layer="91"/>
+<wire x1="73.66" y1="92.71" x2="73.66" y2="73.66" width="0.1524" layer="91"/>
+<pinref part="R5" gate="G$1" pin="1"/>
+<wire x1="73.66" y1="73.66" x2="64.77" y2="73.66" width="0.1524" layer="91"/>
 </segment>
 </net>
@@
 </segment>
 </net>
+<net name="N$5" class="0">
+<segment>
+<pinref part="R5" gate="G$1" pin="2"/>
+<pinref part="X3" gate="-1" pin="S"/>
+<wire x1="64.77" y1="83.82" x2="64.77" y2="89.408" width="0.1524" layer="91"/>
+</segment>
+</net>
