File: locker_unit.brd (EAGLE design)
At the start: 58 x 52 mm, 30 parts, among them IC2 7805T, J1 RJ11, J2 RJ11, Q2 8 MHz, Q4 BC547, U1 PIC16F1705-X/PDIP

Commit message: Edit whole layout, add external LED header. Should be the final version.
Parts:
- removed LED1: RED, SparkFun-LED:LED5MM
- removed LED2: GREEN, SparkFun-LED:LED5MM
- removed R2: 220, SparkFun-Passives:AXIAL-0.3
- added X3: (no value), Locker-custom:KK-156-2
- Q2: device crystal:HC49U70 -> SparkFun-FreqCtrl:HC49US
- moved X2 48.9 mm to (49.9, 40.0)
- moved R1 45.5 mm to (52.4, 6.03), turned to 270 degrees
- moved R5 44.8 mm to (49.8, 14.9)
- moved R8 44.6 mm to (48.7, 6.03), turned to 270 degrees
- moved J1 43.2 mm to (7.63, 7.90)
- moved J2 43.2 mm to (7.63, 44.0)
- moved D2 39.4 mm to (46.7, 38.0)
- moved U$3 38.9 mm to (12.4, 28.9), turned to 180 degrees
- moved R4 38.3 mm to (56.5, 11.7)
- moved R9 33.2 mm to (16.4, 42.5)
- moved D1 31.7 mm to (50.0, 35.5), turned to 0 degrees
- moved C9 31.5 mm to (33.7, 5.08), flipped to the bottom, turned to 90 degrees
- moved JP4 29.6 mm to (19.4, 35.8), turned to 180 degrees
- moved C1 28.0 mm to (16.2, 31.8), turned to 180 degrees
- moved C10 27.0 mm to (25.4, 28.3)
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Connections:
- removed net N$7: LED2.K, R5.P$2
- net GND: no longer R2.P$1, R5.P$1
- net N$12: now also X3.2; no longer LED2.A
- net N$2: now also R5.P$1; no longer LED1.A
- net N$5: now also R5.P$2, X3.1; no longer LED1.K, R2.P$2
Routing:
- net 12V: track 32.2 -> 89.1 mm, vias 0 -> 2
- net CANL: track 27.3 -> 64.6 mm
- net N$12: track 7.54 -> 41.8 mm, vias 0 -> 2
- net N$16: track 21.6 -> 53.4 mm, vias 0 -> 2
- net N$5: track 3.96 -> 33.7 mm, vias 0 -> 2
- net TXCAN: track 33.2 -> 3.96 mm
- net 5V: track 124.9 -> 148.3 mm, vias 0 -> 2
- net N$3: track 24.7 -> 47.7 mm
- net CANH: track 62.3 -> 50.7 mm
- net N$6: track 0.00 -> 10.3 mm
- net LOCK_CTRL: track 15.2 -> 24.5 mm
- net N$17: track 3.39 -> 11.8 mm
- net RXCAN: track 3.93 -> 10.9 mm
- net N$2: track 9.40 -> 3.11 mm
- net N$7: track 6.13 -> 0.00 mm
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- added copper zone on layer 1, net GND
Other:
- outline, holes or cut-outs redrawn

Commit message: Eagle edit?
Parts:
- moved D2 1.27 mm to (47.9, 38.0)
Changed lines of the file:
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@@
 <setting verticaltext="up"/>
 </settings>
-<grid distance="0.05" unitdist="inch" unit="inch" style="lines" multiple="1" display="no" altdistance="0.000000123031" altunitdist="inch" altunit="inch"/>
+<grid distance="0.05" unitdist="inch" unit="inch" style="lines" multiple="1" display="no" altdistance="0.025" altunitdist="inch" altunit="inch"/>
 <layers>
-<layer number="1" name="Top" color="4" fill="1" visible="yes" active="yes"/>
+<layer number="1" name="Top" color="4" fill="1" visible="no" active="yes"/>
 <layer number="2" name="Route2" color="1" fill="3" visible="no" active="no"/>
 <layer number="3" name="Route3" color="4" fill="3" visible="no" active="no"/>
@@
 <layer number="17" name="Pads" color="2" fill="1" visible="yes" active="yes"/>
 <layer number="18" name="Vias" color="2" fill="1" visible="yes" active="yes"/>
-<layer number="19" name="Unrouted" color="6" fill="1" visible="yes" active="yes"/>
+<layer number="19" name="Unrouted" color="6" fill="1" visible="no" active="yes"/>
 <layer number="20" name="Dimension" color="15" fill="1" visible="yes" active="yes"/>
-<layer number="21" name="tPlace" color="7" fill="1" visible="yes" active="yes"/>
-<layer number="22" name="bPlace" color="7" fill="1" visible="yes" active="yes"/>
-<layer number="23" name="tOrigins" color="15" fill="1" visible="yes" active="yes"/>
-<layer number="24" name="bOrigins" color="15" fill="1" visible="yes" active="yes"/>
-<layer number="25" name="tNames" color="7" fill="1" visible="yes" active="yes"/>
-<layer number="26" name="bNames" color="7" fill="1" visible="yes" active="yes"/>
-<layer number="27" name="tValues" color="7" fill="1" visible="yes" active="yes"/>
-<layer number="28" name="bValues" color="7" fill="1" visible="yes" active="yes"/>
+<layer number="21" name="tPlace" color="7" fill="1" visible="no" active="yes"/>
+<layer number="22" name="bPlace" color="7" fill="1" visible="no" active="yes"/>
+<layer number="23" name="tOrigins" color="15" fill="1" visible="no" active="yes"/>
+<layer number="24" name="bOrigins" color="15" fill="1" visible="no" active="yes"/>
+<layer number="25" name="tNames" color="7" fill="1" visible="no" active="yes"/>
+<layer number="26" name="bNames" color="7" fill="1" visible="no" active="yes"/>
+<layer number="27" name="tValues" color="7" fill="1" visible="no" active="yes"/>
+<layer number="28" name="bValues" color="7" fill="1" visible="no" active="yes"/>
 <layer number="29" name="tStop" color="7" fill="3" visible="no" active="yes"/>
 <layer number="30" name="bStop" color="7" fill="6" visible="no" active="yes"/>
@@
 <layer number="43" name="vRestrict" color="2" fill="10" visible="no" active="yes"/>
 <layer number="44" name="Drills" color="7" fill="1" visible="no" active="yes"/>
-<layer number="45" name="Holes" color="7" fill="1" visible="yes" active="yes"/>
+<layer number="45" name="Holes" color="7" fill="1" visible="no" active="yes"/>
 <layer number="46" name="Milling" color="3" fill="1" visible="no" active="yes"/>
 <layer number="47" name="Measures" color="7" fill="1" visible="no" active="yes"/>
@@
 <attribute name="OC_FARNELL" value="unknown" x="49.8525" y="40.005" size="1.778" layer="27" display="off"/>
 </element>
-<element name="D2" library="diode" package="DO41-10" value="1N4004" x="46.6725" y="38.023409375"/>
+<element name="D2" library="diode" package="DO41-10" value="1N4004" x="47.9425" y="38.023409375"/>
 <element name="X3" library="Locker-custom" package="KK-156-2" value="" x="40.64" y="40.005">
 <attribute name="OC_NEWARK" value="unknown" x="40.64" y="40.005" size="1.778" layer="27" display="off"/>
@@
 <wire x1="31.5595" y1="32.4485" x2="30.6705" y2="33.3375" width="0.381" layer="16"/>
 <wire x1="31.5595" y1="32.4485" x2="31.75" y2="32.385" width="0.381" layer="16"/>
-<wire x1="30.6705" y1="40.4495" x2="37.7825" y2="47.5615" width="0.381" layer="16"/>
-<wire x1="37.7825" y1="47.5615" x2="38.6715" y2="48.4505" width="0.381" layer="16"/>
-<wire x1="30.6705" y1="38.6715" x2="30.6705" y2="40.4495" width="0.381" layer="16"/>
-<wire x1="38.6715" y1="48.4505" x2="38.085" y2="48.6975" width="0.381" layer="16"/>
+<wire x1="30.6705" y1="38.6715" x2="30.6705" y2="39.8145" width="0.381" layer="16"/>
 <wire x1="4.445" y1="35.1155" x2="5.334" y2="35.1155" width="0.381" layer="16"/>
 <wire x1="2.667" y1="36.8935" x2="4.445" y2="35.1155" width="0.381" layer="16"/>
 <wire x1="2.667" y1="38.227" x2="2.667" y2="36.8935" width="0.381" layer="16"/>
 <wire x1="35.1155" y1="50.2285" x2="12.1285" y2="50.2285" width="0.381" layer="16"/>
-<wire x1="37.7825" y1="47.5615" x2="35.1155" y2="50.2285" width="0.381" layer="16"/>
 <wire x1="5.334" y1="35.1155" x2="5.725" y2="35.1075" width="0.381" layer="16"/>
 <wire x1="9.535" y1="16.7875" x2="9.535" y2="19.695" width="0.4064" layer="16"/>
@@
 <wire x1="30.348" y1="37.1525" x2="30.6705" y2="36.83" width="0.4064" layer="16"/>
 <wire x1="2.667" y1="38.227" x2="12.1285" y2="50.2285" width="0.4064" layer="16"/>
+<wire x1="35.1155" y1="50.2285" x2="35.56" y2="50.2285" width="0.4064" layer="16"/>
+<wire x1="35.56" y1="50.2285" x2="36.554" y2="50.2285" width="0.4064" layer="16"/>
+<wire x1="36.554" y1="50.2285" x2="38.085" y2="48.6975" width="0.4064" layer="16"/>
+<wire x1="30.6705" y1="39.8145" x2="30.9245" y2="39.8145" width="0.4064" layer="16"/>
+<wire x1="30.9245" y1="39.8145" x2="35.56" y2="44.45" width="0.4064" layer="16"/>
+<wire x1="35.56" y1="44.45" x2="35.56" y2="50.2285" width="0.4064" layer="16"/>
 </signal>
 <signal name="LOCK_CTRL">
@@
 <contactref element="X2" pad="1"/>
 <contactref element="D2" pad="C"/>
-<wire x1="36.8935" y1="38.227" x2="33.782" y2="38.227" width="0.381" layer="16"/>
-<wire x1="38.227" y1="36.8935" x2="36.8935" y2="38.227" width="0.381" layer="16"/>
-<wire x1="40.4495" y1="36.8935" x2="38.227" y2="36.8935" width="0.381" layer="16"/>
-<wire x1="41.3385" y1="37.7825" x2="40.4495" y2="36.8935" width="0.381" layer="16"/>
+<wire x1="35.6235" y1="38.227" x2="33.782" y2="38.227" width="0.381" layer="16"/>
+<wire x1="36.957" y1="36.8935" x2="35.6235" y2="38.227" width="0.381" layer="16"/>
+<wire x1="40.4495" y1="36.8935" x2="36.957" y2="36.8935" width="0.381" layer="16"/>
 <wire x1="33.782" y1="38.227" x2="33.005" y2="38.5375" width="0.381" layer="16"/>
-<wire x1="41.3385" y1="37.7825" x2="41.5925" y2="38.023409375" width="0.381" layer="16"/>
 <wire x1="54.483" y1="41.3385" x2="54.483" y2="42.2275" width="0.381" layer="16"/>
 <wire x1="53.1495" y1="40.005" x2="54.483" y2="41.3385" width="0.381" layer="16"/>
-<wire x1="43.561" y1="40.005" x2="53.1495" y2="40.005" width="0.381" layer="16"/>
-<wire x1="41.783" y1="38.227" x2="43.561" y2="40.005" width="0.381" layer="16"/>
 <wire x1="54.483" y1="42.2275" x2="54.8525" y2="42.305" width="0.381" layer="16"/>
-<wire x1="41.783" y1="38.227" x2="41.5925" y2="38.023409375" width="0.381" layer="16"/>
+<wire x1="40.4495" y1="36.8935" x2="41.732590625" y2="36.8935" width="0.4064" layer="16"/>
+<wire x1="41.732590625" y1="36.8935" x2="42.8625" y2="38.023409375" width="0.4064" layer="16"/>
+<wire x1="42.8625" y1="38.023409375" x2="44.844090625" y2="40.005" width="0.4064" layer="16"/>
+<wire x1="44.844090625" y1="40.005" x2="53.1495" y2="40.005" width="0.4064" layer="16"/>
 </signal>
 <signal name="N$6">
